Commit message: Rename package name to prometheus_sim

File: urdf/prometheus_sim.urdf (robot description, URDF)
Before this commit: robot prometheus_basic, 13 links, 12 joints
Links:
- link fixed_head_link: geometry collision mesh filename=package://prometheus_sim/meshes/low_poly/FIXED_HEAD_LINK_LO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; visual mesh filename=package://prometheus_sim/meshes/mid_poly/FIXED_HEAD_LINK_MI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
- link fixed_left_arm_link: geometry collision mesh filename=package://prometheus_sim/meshes/low_poly/FIXED_LEFT_ARM_LIN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; visual mesh filename=package://prometheus_sim/meshes/mid_poly/FIXED_LEFT_ARM_LIN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
- link right_DOF1_link: geometry collision mesh filename=package://prometheus_sim/meshes/low_poly/LINK_DOF1_RIGHT_AR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; visual mesh filename=package://prometheus_sim/meshes/mid_poly/LINK_DOF1_RIGHT_AR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
- link right_DOF2_link: geometry collision mesh filename=package://prometheus_sim/meshes/low_poly/LINK_DOF2_RIGHT_AR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; visual mesh filename=package://prometheus_sim/meshes/mid_poly/LINK_DOF2_RIGHT_AR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
- link right_DOF3_link: geometry collision mesh filename=package://prometheus_sim/meshes/low_poly/LINK_DOF3_RIGHT_AR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; visual mesh filename=package://prometheus_sim/meshes/mid_poly/LINK_DOF3_RIGHT_AR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
- link right_DOF4_link: geometry collision mesh filename=package://prometheus_sim/meshes/low_poly/LINK_DOF4_RIGHT_AR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; visual mesh filename=package://prometheus_sim/meshes/mid_poly/LINK_DOF4_RIGHT_AR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
- link right_DOF5_link: geometry collision mesh filename=package://prometheus_sim/meshes/low_poly/LINK_DOF5_RIGHT_AR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; visual mesh filename=package://prometheus_sim/meshes/mid_poly/LINK_DOF5_RIGHT_AR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
- link right_DOF6_link: geometry collision mesh filename=package://prometheus_sim/meshes/low_poly/LINK_DOF6_WITH_HAN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; visual mesh filename=package://prometheus_sim/meshes/mid_poly/LINK_DOF6_WITH_HAN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
- link torso_ref_origin_link: geometry collision mesh filename=package://prometheus_sim/meshes/low_poly/LINK_TORSO_REF_ORI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; visual mesh filename=package://prometheus_sim/meshes/mid_poly/LINK_TORSO_REF_ORI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
- link torso_yaw_link: geometry collision mesh filename=package://prometheus_sim/meshes/low_poly/LINK_TORSO_YAW_LOW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; visual mesh filename=package://prometheus_sim/meshes/mid_poly/LINK_TORSO_YAW_MID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
